Commit message: updated urdf

File: assets/qarm-community/qarm_with_gripper.urdf (robot description, URDF)
Before this commit: robot QARM, 11 links, 10 joints
Links:
- link BICEP: geometry collision cylinder length=0.35 radius=0.05; visual mesh filename=meshes/BICEP.STL
- link END-EFFECTOR: geometry visual mesh filename=meshes/END-EFFECTOR.STL
- link FOREARM: geometry collision cylinder length=0.24 radius=0.03; visual mesh filename=meshes/FOREARM.STL
- link Link1A: geometry collision box size=0.006411377 0.01555569 0.03100051; collision box size=0.01421403 0.01688009 0.0343732
- link Link1B: geometry collision box size=0.01721035 0.0185371 0.01886072; collision box size=0.02039559 0.02205 0.04227039
- link Link2A: geometry collision box size=0.0217 0.02303058 0.05918772; visual mesh filename=meshes/LINK2A.STL
- link Link2B: geometry collision box size=0.0217 0.02303058 0.05918772; visual mesh filename=meshes/LINK2B.STL
- link YAW: geometry collision box size=0.05 0.16 0.07; visual mesh filename=meshes/YAW.STL
- link base_link: geometry collision box size=0.3 0.35 0.1; visual mesh filename=meshes/base_link.STL
- link gripper_base_link: geometry collision box size=0.04 0.08 0.09; visual mesh filename=meshes/gripper_base_link.STL
Joints:
- joint WRIST: limit lower=-3.010 upper=3.010 effort=0 velocity=0 -> lower=-3.01 upper=3.01 effort=0 velocity=0
